File: LX780_Delta-fixed/NE_Delta.kicad_pcb (KiCad board)
At the start: 2 copper layers, 379.1 x 273.4 mm, 185 parts, among them IC1 74LS00, IC10 4164, IC11 4164, IC12 4164, IC13 4164, IC14 4164, IC15 4164, IC16 4164, IC17 4164, IC18 4164, IC19 4164, IC2 74LS04, IC20 4164, IC21 4164, IC22 4164, IC23 4164, IC24 74LS245, IC25 74LS374, IC26 74LS374, IC27 2764, IC28 2764, IC29 GAL16V8, IC3 74LS02, IC30 74LS74, IC31 74LS153, IC32 74LS153, IC33 74LS153, IC34 74LS153, IC35 74LS244, IC36 74LS244, IC37 6502, IC38 74LS245, IC39 74LS125, IC4 74LS138, IC40 74LS04, IC41 74LS173, IC42 GAL16V8, IC43 74LS20, IC44 74LS00, IC45 GAL16V8, IC46 74LS74, IC47 GAL16V8, IC48 GAL16V8, IC49 74LS165, IC5 74LS04, IC50 74LS374, IC51 74LS02, IC52 74LS374, IC53 74LS157, IC54 GAL16V8, IC55 2732, IC56 74LS153, IC57 GAL16V8, IC58 74LS259, IC59 74LS283, IC6 74LS32, IC60 74LS00, IC61 74LS157, IC62 6545, IC63 74LS251, IC64 74LS259, IC65 74LS251, IC66 74LS251, IC67 NE556, IC68 NE556, IC69 74LS138, IC7 74LS138, IC70 μA741, IC71 74LS74, IC72 74LS244, IC73 NE556, IC8 4164, IC9 4164, J1 Tape IN, J2 Tape OUT, P1 Jumper_3_Bridged12, P2 Jumper_3_Bridged12, P3 Jumper_3_Bridged12, P4 Jumper_3_Bridged12, P5 SolderJumper_2_Open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

Commit message: update
Connections:
- IC5 pad 9: Net-(IC41-Q2) -> Net-(IC41-Q0)
- IC63 pad 2: Net-(IC41-Q0) -> Net-(IC41-Q2)
Routing:
- net Net-(IC41-Q0): track 210.7 -> 354.0 mm, vias 8 -> 11
- net Net-(IC41-Q2): track 342.5 -> 208.0 mm, vias 11 -> 8
