File: LX780_Delta-fixed/NE_Delta.kicad_sch (KiCad schematic)
At the start: 45 parts, among them IC1 74LS00, IC2 74LS04, IC3 74LS02, IC30 74LS74, IC39 74LS125, IC40 74LS04, IC43 74LS20, IC44 74LS00, IC46 74LS74, IC5 74LS04, IC51 74LS02, IC6 74LS32, IC60 74LS00, IC71 74LS74

Commit message: update
Connections:
- net NOT_READ_EN_G renamed NOT_BANK_SEL_G
- net READ_EN_G renamed BANK_SEL_G
Changed lines of the file:
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@@
 		)
 	)
-	(global_label "READ_EN_G"
+	(global_label "BANK_SEL_G"
 		(shape input)
 		(at 48.26 76.2 180)
@@
 		)
 		(property "Intersheetrefs" "${INTERSHEET_REFS}"
-			(at 34.8125 76.2 0)
+			(at 33.7239 76.2 0)
 			(effects
 				(font
@@
 		)
 	)
-	(global_label "NOT_READ_EN_G"
+	(global_label "NOT_BANK_SEL_G"
 		(shape output)
 		(at 78.74 76.2 0)
@@
 		)
 		(property "Intersheetrefs" "${INTERSHEET_REFS}"
-			(at 96.7837 76.2 0)
+			(at 97.8723 76.2 0)
 			(effects
 				(font
