File: LX780_Delta-fixed/io.kicad_sch (KiCad schematic)
At the start: 84 parts, among them IC1 74LS00, IC2 74LS04, IC30 74LS74, IC40 74LS04, IC49 74LS165, IC5 74LS04, IC50 74LS374, IC51 74LS02, IC52 74LS374, IC53 74LS157, IC54 GAL16V8, IC55 2732, IC56 74LS153, IC57 GAL16V8, IC58 74LS259, IC59 74LS283, IC6 74LS32, IC60 74LS00, IC61 74LS157, IC62 6545, IC63 74LS251, IC64 74LS259, IC65 74LS251, IC66 74LS251, IC67 NE556, IC68 NE556, IC69 74LS138, IC70 μA741, IC71 74LS74, IC72 74LS244, IC73 NE556, J1 Tape IN, J2 Tape OUT, P3 Jumper_3_Bridged12, P4 Jumper_3_Bridged12, P5 SolderJumper_2_Open, P6 Jumper_3_Bridged12, P7 Jumper_3_Bridged12, P8 Jumper_3_Bridged12

Commit message: update
Connections:
- net BANK_SEL_G renamed READ_EN_G
- net NOT_READ_EN_G renamed NOT_BANK_SEL_G
Changed lines of the file:
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@@
 		)
 	)
-	(global_label "BANK_SEL_G"
+	(global_label "READ_EN_G"
 		(shape output)
 		(at 81.28 344.17 0)
@@
 		)
 		(property "Intersheetrefs" "${INTERSHEET_REFS}"
-			(at 95.8161 344.17 0)
+			(at 94.7275 344.17 0)
 			(effects
 				(font
@@
 		)
 	)
-	(global_label "NOT_READ_EN_G"
+	(global_label "NOT_BANK_SEL_G"
 		(shape input)
 		(at 88.9 349.25 0)
@@
 		)
 		(property "Intersheetrefs" "${INTERSHEET_REFS}"
-			(at 106.9437 349.25 0)
-			(effects
-				(font
+			(at 108.0323 349.25 0)
+			(effects
+				(font
